File: motorsystem_test.brd (EAGLE design)
At the start: 100 x 80 mm, 5 parts

Commit message: 図面作成
Parts:
- added C3: 0.1u, rcl:C025-030X050
- added IC2: (no value), user_ic:DIL8
- added R2: 120, rcl:0207/2V
- added SW1: TOGURUSUIITI, user_swich:TOGURUSUIITI
- added U$3: NUCLEO-F303K8, user_ic:NUCLEO-NANO
- C1: value (none) -> 0.47u
- C2: value (none) -> 0.22u
- moved C2 17.5 mm to (16.5, 22.9), turned to 180 degrees
- moved U$2 16.1 mm to (45.7, 15.2)
- moved IC1 13.6 mm to (15.1, 20.3), turned to 0 degrees
- moved U$1 11.4 mm to (17.8, 10.0), turned to 180 degrees
- moved C1 3.86 mm to (13.8, 12.7), turned to 0 degrees
Connections:
- removed net N$3: U$2.P$5
- removed net N$4: U$2.P$6
- new net CANH: IC2.PIN6, R2.2, U$2.P$5
- new net CANL: IC2.PIN7, R2.1, U$2.P$6
- new net CAN_RX: IC2.PIN4, U$3.P$13
- new net CAN_TX: IC2.PIN1, U$3.P$5
- new net N$1: SW1.2, SW1.C, U$1.P$2
- new net N$7: IC2.PIN8, U$3.P$17
- net +12V: now also SW1.1; no longer U$1.P$2
- net +5V: now also C3.1, IC2.PIN3, IC2.PIN5, U$3.P$27
- net GND: now also C3.2, IC2.PIN2, U$3.P$29
Routing:
- net GND: track 0.00 -> 114.7 mm
- net +12V: track 0.00 -> 94.3 mm
- net +5V: track 0.00 -> 89.0 mm
- net N$7: track 0.00 -> 43.2 mm
- net CAN_RX: track 0.00 -> 30.5 mm
- net CAN_TX: track 0.00 -> 12.7 mm
- net N$1: track 0.00 -> 12.6 mm
- net CANL: track 0.00 -> 11.2 mm
- net CANH: track 0.00 -> 7.62 mm

Commit message: vin
Parts:
- turned R2 to 90 degrees
Connections:
- net +12V: now also U$3.P$30
- net +5V: no longer IC2.PIN5, U$3.P$27
- net CANH: now also IC2.PIN7; no longer IC2.PIN6
- net CANL: now also IC2.PIN6; no longer IC2.PIN7
- net GND: now also IC2.PIN8
- net N$7: now also IC2.PIN5; no longer IC2.PIN8
Routing:
- net N$7: track 43.2 -> 55.9 mm
- net GND: track 114.7 -> 123.3 mm
- net +5V: track 89.0 -> 81.3 mm
- net CANL: track 11.2 -> 13.8 mm
- net CANH: track 7.62 -> 10.2 mm
Changed lines of the file:
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@@
 <attribute name="VALUE" x="5.08" y="5.08" size="1.27" layer="27"/>
 </element>
-<element name="R2" library="rcl" library_urn="urn:adsk.eagle:library:334" package="0207/2V" package3d_urn="urn:adsk.eagle:package:23490/1" value="120" x="38.1" y="16.51" smashed="yes" rot="R270">
-<attribute name="NAME" x="39.116" y="16.5608" size="1.27" layer="25" ratio="10" rot="R270"/>
-<attribute name="POPULARITY" value="17" x="38.1" y="16.51" size="1.778" layer="27" rot="R270" display="off"/>
-<attribute name="SPICEPREFIX" value="R" x="38.1" y="16.51" size="1.778" layer="27" rot="R270" display="off"/>
-<attribute name="VALUE" x="35.8648" y="16.5608" size="1.27" layer="27" ratio="10" rot="R270"/>
+<element name="R2" library="rcl" library_urn="urn:adsk.eagle:library:334" package="0207/2V" package3d_urn="urn:adsk.eagle:package:23490/1" value="120" x="38.1" y="16.51" smashed="yes" rot="R90">
+<attribute name="NAME" x="37.084" y="16.4592" size="1.27" layer="25" ratio="10" rot="R90"/>
+<attribute name="POPULARITY" value="17" x="38.1" y="16.51" size="1.778" layer="27" rot="R90" display="off"/>
+<attribute name="SPICEPREFIX" value="R" x="38.1" y="16.51" size="1.778" layer="27" rot="R90" display="off"/>
+<attribute name="VALUE" x="40.3352" y="16.4592" size="1.27" layer="27" ratio="10" rot="R90"/>
 </element>
 </elements>
@@
 <wire x1="7.62" y1="15.24" x2="10.16" y2="15.24" width="0.1524" layer="16"/>
 <wire x1="10.16" y1="15.24" x2="10.16" y2="12.7" width="0.1524" layer="16"/>
+<contactref element="U$3" pad="P$30"/>
+<wire x1="12.573" y1="17.78" x2="12.7" y2="43.18" width="0" layer="19" extent="1-1"/>
 </signal>
 <signal name="+5V">
@@
 <contactref element="U$2" pad="P$10"/>
 <contactref element="C2" pad="1"/>
-<contactref element="U$3" pad="P$27"/>
 <contactref element="IC2" pad="PIN3"/>
-<contactref element="IC2" pad="PIN5"/>
 <contactref element="C3" pad="1"/>
 <wire x1="27.94" y1="15.24" x2="25.4" y2="15.24" width="0.1524" layer="16"/>
 <wire x1="25.4" y1="15.24" x2="25.4" y2="10.16" width="0.1524" layer="16"/>
 <wire x1="25.4" y1="10.16" x2="35.56" y2="10.16" width="0.1524" layer="16"/>
-<wire x1="35.56" y1="10.16" x2="35.56" y2="12.7" width="0.1524" layer="16"/>
 <wire x1="45.72" y1="10.16" x2="43.18" y2="10.16" width="0.1524" layer="16"/>
 <wire x1="43.18" y1="10.16" x2="35.56" y2="10.16" width="0.1524" layer="16"/>
@@
 <wire x1="10.16" y1="25.4" x2="10.16" y2="38.1" width="0.1524" layer="16"/>
 <wire x1="10.16" y1="38.1" x2="20.32" y2="38.1" width="0.1524" layer="16"/>
-<wire x1="20.32" y1="38.1" x2="20.32" y2="43.18" width="0.1524" layer="16"/>
 <wire x1="17.78" y1="22.86" x2="17.78" y2="25.4" width="0.1524" layer="16"/>
 <wire x1="17.78" y1="22.86" x2="17.78" y2="17.907" width="0.1524" layer="16"/>
@@
 <wire x1="15.24" y1="40.64" x2="15.24" y2="43.18" width="0.1524" layer="16"/>
 <wire x1="15.24" y1="22.86" x2="7.62" y2="22.86" width="0.1524" layer="16"/>
+<contactref element="IC2" pad="PIN8"/>
+<wire x1="35.56" y1="20.32" x2="33.02" y2="17.78" width="0.1524" layer="1"/>
+<wire x1="33.02" y1="17.78" x2="27.94" y2="17.78" width="0.1524" layer="1"/>
 <wire x1="15.113" y1="12.7" x2="15.33" y2="7.683" width="0" layer="19" extent="1-1"/>
 </signal>
 <signal name="CANH">
 <contactref element="U$2" pad="P$5"/>
-<contactref element="IC2" pad="PIN6"/>
+<contactref element="IC2" pad="PIN7"/>
 <contactref element="R2" pad="2"/>
-<wire x1="35.56" y1="15.24" x2="38.1" y2="15.24" width="0.1524" layer="16"/>
-<wire x1="38.1" y1="15.24" x2="43.18" y2="15.24" width="0.1524" layer="16"/>
+<wire x1="35.56" y1="17.78" x2="38.1" y2="17.78" width="0.1524" layer="16"/>
+<wire x1="38.1" y1="17.78" x2="40.64" y2="17.78" width="0.1524" layer="16"/>
+<wire x1="40.64" y1="17.78" x2="40.64" y2="15.24" width="0.1524" layer="16"/>
+<wire x1="40.64" y1="15.24" x2="43.18" y2="15.24" width="0.1524" layer="16"/>
 </signal>
 <signal name="CANL">
 <contactref element="U$2" pad="P$6"/>
-<contactref element="IC2" pad="PIN7"/>
-<wire x1="45.0332875" y1="15.24" x2="45.72" y2="15.24" width="0.1524" layer="16"/>
-<wire x1="44.0396875" y1="16.2336" x2="45.0332875" y2="15.24" width="0.1524" layer="16"/>
+<contactref element="IC2" pad="PIN6"/>
 <contactref element="R2" pad="1"/>
-<wire x1="39.6464" y1="16.2336" x2="44.0396875" y2="16.2336" width="0.1524" layer="16"/>
-<wire x1="39.6464" y1="16.2336" x2="38.1" y2="17.78" width="0.1524" layer="16"/>
-<wire x1="38.1" y1="17.78" x2="35.56" y2="17.78" width="0.1524" layer="16"/>
+<wire x1="38.1" y1="15.24" x2="35.56" y2="15.24" width="0.1524" layer="16"/>
+<wire x1="45.72" y1="15.24" x2="44.1736" y2="13.6936" width="0.1524" layer="16"/>
+<wire x1="44.1736" y1="13.6936" x2="42.3203125" y2="13.6936" width="0.1524" layer="16"/>
+<wire x1="42.3203125" y1="13.6936" x2="41.3267125" y2="12.7" width="0.1524" layer="16"/>
+<wire x1="38.1" y1="12.7" x2="38.1" y2="15.24" width="0.1524" layer="16"/>
+<wire x1="41.3267125" y1="12.7" x2="38.1" y2="12.7" width="0.1524" layer="16"/>
 </signal>
 <signal name="CAN_RX">
 <contactref element="U$3" pad="P$13"/>
 <contactref element="IC2" pad="PIN4"/>
-<wire x1="27.94" y1="12.7" x2="33.02" y2="12.7" width="0.1524" layer="16"/>
-<wire x1="33.02" y1="12.7" x2="33.02" y2="25.4" width="0.1524" layer="16"/>
-<wire x1="33.02" y1="25.4" x2="43.18" y2="25.4" width="0.1524" layer="16"/>
+<wire x1="27.94" y1="12.7" x2="30.48" y2="12.7" width="0.1524" layer="16"/>
+<wire x1="30.48" y1="12.7" x2="30.48" y2="25.4" width="0.1524" layer="16"/>
+<wire x1="30.48" y1="25.4" x2="43.18" y2="25.4" width="0.1524" layer="16"/>
 <wire x1="43.18" y1="25.4" x2="43.18" y2="27.94" width="0.1524" layer="16"/>
 </signal>
@@
 </signal>
 <signal name="N$7">
-<contactref element="IC2" pad="PIN8"/>
+<contactref element="IC2" pad="PIN5"/>
 <contactref element="U$3" pad="P$17"/>
 <wire x1="45.72" y1="43.18" x2="45.72" y2="35.56" width="0.1524" layer="16"/>
 <wire x1="45.72" y1="35.56" x2="50.8" y2="35.56" width="0.1524" layer="16"/>
 <wire x1="50.8" y1="35.56" x2="50.8" y2="22.86" width="0.1524" layer="16"/>
-<wire x1="50.8" y1="22.86" x2="35.56" y2="22.86" width="0.1524" layer="16"/>
-<wire x1="35.56" y1="22.86" x2="35.56" y2="20.32" width="0.1524" layer="16"/>
+<wire x1="50.8" y1="22.86" x2="33.02" y2="22.86" width="0.1524" layer="16"/>
+<wire x1="33.02" y1="22.86" x2="33.02" y2="12.7" width="0.1524" layer="16"/>
+<wire x1="33.02" y1="12.7" x2="35.56" y2="12.7" width="0.1524" layer="16"/>
 </signal>
 <signal name="N$1">
