File: motorsystem_test.sch (EAGLE design)
At the start: 5 parts

Commit message: 図面作成
Parts:
- added C3: 0.1u, rcl:C-EU025-030X050
- added IC2: (no value), user_ic:MCP2562
- added R2: 120, rcl:R-EU_0207/2V
- added SW1: TOGURUSUIITI, user_swich:TOGURUSUIITI
- added U$3: NUCLEO-F303K8, user_ic:NUCLEO-F303K8
- C1: value (none) -> 0.47u
- C2: value (none) -> 0.22u
Connections:
- removed net N$3: U$2.P$5
- removed net N$4: U$2.P$6
- new net CANH: IC2.CANH, R2.2, U$2.P$5
- new net CANL: IC2.CANL, R2.1, U$2.P$6
- new net CAN_RX: IC2.RXD, U$3.PA11
- new net CAN_TX: IC2.TXD, U$3.PA12
- new net N$1: SW1.2, SW1.C, U$1.PIN2
- new net N$7: IC2.VIO, U$3.+3V3
- net +12V: now also SW1.1; no longer U$1.PIN2
- net +5V: now also C3.1, IC2.STBY, IC2.VDD, U$3.+5V
- net GND: now also C3.2, IC2.VSS, U$3.GND@2

Commit message: vin
Connections:
- net +12V: now also U$3.VIN
- net +5V: no longer IC2.STBY, U$3.+5V
- net GND: now also IC2.STBY
Changed lines of the file:
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@@
 <part name="C2" library="rcl" library_urn="urn:adsk.eagle:library:334" deviceset="C-EU" device="025-030X050" package3d_urn="urn:adsk.eagle:package:23631/1" value="0.22u"/>
 <part name="U$3" library="user_ic" deviceset="NUCLEO-F303K8" device=""/>
-<part name="P+5" library="supply1" library_urn="urn:adsk.eagle:library:371" deviceset="+5V" device=""/>
 <part name="IC2" library="user_ic" deviceset="MCP2562" device=""/>
 <part name="GND3" library="supply1" library_urn="urn:adsk.eagle:library:371" deviceset="GND" device=""/>
@@
 </instance>
 <instance part="U$3" gate="G$1" x="-10.16" y="-15.24" smashed="yes"/>
-<instance part="P+5" gate="1" x="15.24" y="12.7" smashed="yes">
-<attribute name="VALUE" x="12.7" y="7.62" size="1.778" layer="96" rot="R90"/>
-</instance>
 <instance part="IC2" gate="G$1" x="88.9" y="-12.7" smashed="yes"/>
 <instance part="GND3" gate="1" x="66.04" y="-27.94" smashed="yes">
@@
 <pinref part="P+2" gate="1" pin="+12V"/>
 <wire x1="12.7" y1="71.12" x2="12.7" y2="63.5" width="0.1524" layer="91"/>
-<wire x1="12.7" y1="63.5" x2="33.02" y2="63.5" width="0.1524" layer="91"/>
 <pinref part="IC1" gate="1" pin="IN"/>
 <junction x="12.7" y="71.12"/>
@@
 <wire x1="-5.08" y1="78.74" x2="-5.08" y2="71.12" width="0.1524" layer="91"/>
 <junction x="-5.08" y="71.12"/>
+<wire x1="33.02" y1="63.5" x2="12.7" y2="63.5" width="0.1524" layer="91"/>
+<wire x1="12.7" y1="63.5" x2="12.7" y2="20.32" width="0.1524" layer="91"/>
+<pinref part="U$3" gate="G$1" pin="VIN"/>
+<wire x1="12.7" y1="20.32" x2="5.08" y2="20.32" width="0.1524" layer="91"/>
 </segment>
 <segment>
@@
 </segment>
 <segment>
-<pinref part="U$3" gate="G$1" pin="+5V"/>
-<wire x1="5.08" y1="5.08" x2="15.24" y2="5.08" width="0.1524" layer="91"/>
-<wire x1="15.24" y1="5.08" x2="15.24" y2="10.16" width="0.1524" layer="91"/>
-<pinref part="P+5" gate="1" pin="+5V"/>
-</segment>
-<segment>
 <pinref part="IC2" gate="G$1" pin="VDD"/>
 <wire x1="76.2" y1="-15.24" x2="63.5" y2="-15.24" width="0.1524" layer="91"/>
 <wire x1="63.5" y1="-15.24" x2="63.5" y2="-10.16" width="0.1524" layer="91"/>
 <pinref part="P+6" gate="1" pin="+5V"/>
-<pinref part="IC2" gate="G$1" pin="STBY"/>
-<wire x1="63.5" y1="-10.16" x2="63.5" y2="0" width="0.1524" layer="91"/>
-<wire x1="63.5" y1="0" x2="63.5" y2="2.54" width="0.1524" layer="91"/>
-<wire x1="101.6" y1="-5.08" x2="106.68" y2="-5.08" width="0.1524" layer="91"/>
-<wire x1="106.68" y1="-5.08" x2="106.68" y2="0" width="0.1524" layer="91"/>
-<wire x1="106.68" y1="0" x2="63.5" y2="0" width="0.1524" layer="91"/>
-<junction x="63.5" y="0"/>
+<wire x1="63.5" y1="-10.16" x2="63.5" y2="2.54" width="0.1524" layer="91"/>
 <pinref part="C3" gate="G$1" pin="1"/>
 <wire x1="58.42" y1="-10.16" x2="63.5" y2="-10.16" width="0.1524" layer="91"/>
@@
 <wire x1="58.42" y1="-17.78" x2="66.04" y2="-17.78" width="0.1524" layer="91"/>
 <junction x="66.04" y="-17.78"/>
+<pinref part="IC2" gate="G$1" pin="STBY"/>
+<wire x1="101.6" y1="-5.08" x2="104.14" y2="-5.08" width="0.1524" layer="91"/>
+<wire x1="101.6" y1="-5.08" x2="88.9" y2="-5.08" width="0.1524" layer="91"/>
+<wire x1="88.9" y1="-5.08" x2="88.9" y2="-10.16" width="0.1524" layer="91"/>
+<wire x1="88.9" y1="-10.16" x2="76.2" y2="-10.16" width="0.1524" layer="91"/>
+<junction x="76.2" y="-10.16"/>
 </segment>
 <segment>
